Commit message: Init of aruco detection

File: urdf/robot.xacro (robot description, xacro)
@@ -124,37 +124,17 @@
      <inertial>
         <mass value="0.025"/>
-  	<origin xyz="0 0 0.25" rpy="0 0 0" />
+  	<origin xyz="0 0 0.35" rpy="0 0 0" />
   	<inertia ixx="0.000010279" ixy="0" ixz="0" iyy="0.000010279" iyz="0" izz="0.000007225"/>
      </inertial>
      <collision>
-        <origin xyz="0 0 0.25" rpy="0 0 0"/>
-        <geometry>
-        <box size="0.05 0.05 0.5"/>
+        <origin xyz="0 0 0.35" rpy="0 0 0"/>
+        <geometry>
+        <box size="0.05 0.05 0.7"/>
         </geometry>
      </collision>
      <visual>
-        <origin xyz="0 0 0.25" rpy="0 0 0"/>
-        <geometry>
-        <box size="0.05 0.05 0.5"/>
-        </geometry>
-        <material name="red" />
-     </visual>
-  </link>
-  <link name="arm_link2">
-     <inertial>
-        <mass value="0.025"/>
-  	<origin xyz="0 0 0.25" rpy="0 0 0" />
-  	<inertia ixx="0.000010279" ixy="0" ixz="0" iyy="0.000010279" iyz="0" izz="0.000007225"/>
-     </inertial>
-     <collision>
-        <origin xyz="0 0 0.25" rpy="0 0 0"/>
-        <geometry>
-        <box size="0.05 0.05 0.5"/>
-        </geometry>
-     </collision>
-     <visual>
-        <origin xyz="0 0 0.25" rpy="0 0 0"/>
-        <geometry>
-        <box size="0.05 0.05 0.5"/>
+        <origin xyz="0 0 0.35" rpy="0 0 0"/>
+        <geometry>
+        <box size="0.05 0.05 0.7"/>
         </geometry>
         <material name="red" />
@@ -170,19 +150,9 @@
         <joint_properties damping="1.0" friction="1.0"/>
   </joint>
-  <joint name="arm_joint1" type="revolute">
+  <joint name="arm_joint1" type="fixed">
   	<axis rpy="0 0 0" xyz="0 1 0"/>
   	<origin rpy="0 0 0" xyz="0 0 0.05"/>
   	<parent link="arm_base_link"/>
   	<child link="arm_link1"/>
-  	<limit effort="1000.0" lower="-1.8" upper="1.8" velocity="0.3"/>
-  	<joint_properties damping="1.0" friction="1.0"/>
-  </joint>
-  <joint name="arm_joint2" type="revolute">
-  	<axis rpy="0 0 0" xyz="0 1 0"/>
-  	<origin rpy="0 0 0" xyz="0 0.05 0.45"/>
-  	<parent link="arm_link1"/>
-  	<child link="arm_link2"/>
-  	<limit effort="1000.0" lower="-1.8" upper="1.8" velocity="0.3"/>
-  	<joint_properties damping="1.0" friction="1.0"/>
   </joint>
   <!-- Sensors definition -->
@@ -233,9 +203,11 @@
       </inertial>
   </link>
-  <joint name="camera_joint" type="fixed">
-	<axis xyz="0 1 0" />
-	<origin xyz="0 0 0.525" rpy="0 0 0"/>
-	<parent link="arm_link2"/>
+  <joint name="camera_joint" type="revolute">
+	<axis rpy="0 0 0" xyz="1 0 0" />
+	<origin xyz="0 0 0.725" rpy="0 0 0"/>
+	<parent link="arm_link1"/>
 	<child link="camera_link"/>
+	<limit effort="10000" lower="-3.14" upper="3.14" velocity="0.6"/>
+        <joint_properties damping="1.0" friction="1.0"/>
   </joint>
   <!-- Transission definition -->
@@ -250,20 +222,10 @@
 	</actuator>
   </transmission>
-  <transmission name="arm_joint1_trans">
+  <transmission name="camera_joint_trans">
 	<type>transmission_interface/SimpleTransmission</type>
-	<joint name="arm_joint1">
+	<joint name="camera_joint">
 		<hardwareInterface>hardware_interface/EffortJointInterface</hardwareInterface>
 	</joint>
 	<actuator name="motor2">
-		<hardwareInterface>hardware_interface/EffortJointInterface</hardwareInterface>
-		<mechanicalInterface>1</mechanicalInterface>
-	</actuator>
-  </transmission>
-  <transmission name="arm_joint2_trans">
-	<type>transmission_interface/SimpleTransmission</type>
-	<joint name="arm_joint2">
-		<hardwareInterface>hardware_interface/EffortJointInterface</hardwareInterface>
-	</joint>
-	<actuator name="motor3">
 		<hardwareInterface>hardware_interface/EffortJointInterface</hardwareInterface>
 		<mechanicalInterface>1</mechanicalInterface>

Commit message: Done

File: urdf/robot.xacro (robot description, xacro)
@@ -204,5 +204,5 @@
   </link>
   <joint name="camera_joint" type="revolute">
-	<axis rpy="0 0 0" xyz="1 0 0" />
+	<axis rpy="0 0 0" xyz="0 1 0" />
 	<origin xyz="0 0 0.725" rpy="0 0 0"/>
 	<parent link="arm_link1"/>
